Commit message: Remove rosbridge launch files and add URDF/XACRO files for hexapod model
- Deleted rosbridge.launch and rosbridge.launch.py files as they are no longer needed.
- Added common_properties.xacro to define material properties for the hexapod.
- Introduced hexapod_base.xacro containing the complete URDF description of the hexapod, including links, joints, and transmissions for all legs.
- Created hexapod_base_gazebo.xacro to integrate with Gazebo, including ros2_control plugin and material properties for simulation.

File: hexapod/urdf/hexapod_model.urdf.xacro (robot description, xacro)
@@ -1,680 +1,6 @@
 <?xml version="1.0" ?>
 <robot name="hexapod_model" xmlns:xacro="http://www.ros.org/wiki/xacro">
-<xacro:include filename="$(find hexapod_model_description)/urdf/materials.xacro" />
-<xacro:include filename="$(find hexapod_model_description)/urdf/hexapod_model.gazebo.xacro" />
-<link name="base_link">
-  <inertial>
-    <origin xyz="-0.026500000000020115 0.1853149788824598 0.005671016395165651" rpy="0 0 0"/>
-    <mass value="2.06"/>
-    <inertia ixx="0.009141" iyy="0.006072" izz="0.015206" ixy="-0.0" iyz="0.0" ixz="-0.0"/>
-  </inertial>
-  <visual>
-    <origin xyz="0 0 0" rpy="0 0 0"/>
-    <geometry>
-      <mesh filename="file://$(find hexapod_model_description)/meshes/base_link.stl" scale="0.001 0.001 0.001"/>
-    </geometry>
-    <material name="silver"/>
-  </visual>
-  <collision>
-    <origin xyz="0 0 0" rpy="0 0 0"/>
-    <geometry>
-      <mesh filename="file://$(find hexapod_model_description)/meshes/base_link.stl" scale="0.001 0.001 0.001"/>
-    </geometry>
-  </collision>
-</link>
-<link name="tibia_1_link_1">
-  <inertial>
-    <origin xyz="0.00010740246556076305 -0.06266738282319978 3.191642993887996e-07" rpy="0 0 0"/>
-    <mass value="0.827"/>
-    <inertia ixx="0.002294" iyy="0.000283" izz="0.002521" ixy="-2.0e-05" iyz="-0.0" ixz="-0.0"/>
-  </inertial>
-  <visual>
-    <origin xyz="0.0265 0.0852 -0.000912" rpy="0 0 0"/>
-    <geometry>
-      <mesh filename="file://$(find hexapod_model_description)/meshes/tibia_1_link_1.stl" scale="0.001 0.001 0.001"/>
-    </geometry>
-    <material name="silver"/>
-  </visual>
-  <collision>
-    <origin xyz="0.0265 0.0852 -0.000912" rpy="0 0 0"/>
-    <geometry>
-      <mesh filename="file://$(find hexapod_model_description)/meshes/tibia_1_link_1.stl" scale="0.001 0.001 0.001"/>
-    </geometry>
-  </collision>
-</link>
-<link name="femur_1_link_1">
-  <inertial>
-    <origin xyz="0.0 -0.0477000000000007 3.1916430001611897e-07" rpy="0 0 0"/>
-    <mass value="1.578"/>
-    <inertia ixx="0.002000" iyy="0.000406" izz="0.002148" ixy="0.0" iyz="-0.0" ixz="0.0"/>
-  </inertial>
-  <visual>
-    <origin xyz="0.0265 -0.0102 -0.000912" rpy="0 0 0"/>
-    <geometry>
-      <mesh filename="file://$(find hexapod_model_description)/meshes/femur_1_link_1.stl" scale="0.001 0.001 0.001"/>
-    </geometry>
-    <material name="silver"/>
-  </visual>
-  <collision>
-    <origin xyz="0.0265 -0.0102 -0.000912" rpy="0 0 0"/>
-    <geometry>
-      <mesh filename="file://$(find hexapod_model_description)/meshes/femur_1_link_1.stl" scale="0.001 0.001 0.001"/>
-    </geometry>
-  </collision>
-</link>
-<link name="coxa_1_link_1">
-  <inertial>
-    <origin xyz="1.521040238205984e-13 -0.03676640708236653 -0.010119187749198146" rpy="0 0 0"/>
-    <mass value="0.467"/>
-    <inertia ixx="0.000248" iyy="0.000172" izz="0.000371" ixy="-0.0" iyz="-3.6e-05" ixz="0.0"/>
-  </inertial>
-  <visual>
-    <origin xyz="0.0265 -0.0694 -0.013762" rpy="0 0 0"/>
-    <geometry>
-      <mesh filename="file://$(find hexapod_model_description)/meshes/coxa_1_link_1.stl" scale="0.001 0.001 0.001"/>
-    </geometry>
-    <material name="silver"/>
-  </visual>
-  <collision>
-    <origin xyz="0.0265 -0.0694 -0.013762" rpy="0 0 0"/>
-    <geometry>
-      <mesh filename="file://$(find hexapod_model_description)/meshes/coxa_1_link_1.stl" scale="0.001 0.001 0.001"/>
-    </geometry>
-  </collision>
-</link>
-<link name="tibia_2_link_1">
-  <inertial>
-    <origin xyz="-0.0442362191094724 -0.04438810927594172 3.1916429906462315e-07" rpy="0 0 0"/>
-    <mass value="0.6509579807539126"/>
-    <inertia ixx="0.000998" iyy="0.00103" izz="0.001984" ixy="-0.000792" iyz="-0.0" ixz="-0.0"/>
-  </inertial>
-  <visual>
-    <origin xyz="0.217101 0.006251 -0.000912" rpy="0 0 0"/>
-    <geometry>
-      <mesh filename="file://$(find hexapod_model_description)/meshes/tibia_2_link_1.stl" scale="0.001 0.001 0.001"/>
-    </geometry>
-    <material name="silver"/>
-  </visual>
-  <collision>
-    <origin xyz="0.217101 0.006251 -0.000912" rpy="0 0 0"/>
-    <geometry>
-      <mesh filename="file://$(find hexapod_model_description)/meshes/tibia_2_link_1.stl" scale="0.001 0.001 0.001"/>
-    </geometry>
-  </collision>
-</link>
-<link name="femur_2_link_1">
-  <inertial>
-    <origin xyz="-0.03372863930509079 -0.03372863944813179 3.191642998237815e-07" rpy="0 0 0"/>
-    <mass value="1.2425883897057017"/>
-    <inertia ixx="0.000947" iyy="0.000947" izz="0.001691" ixy="-0.000627" iyz="-0.0" ixz="-0.0"/>
-  </inertial>
-  <visual>
-    <origin xyz="0.149643 -0.061207 -0.000912" rpy="0 0 0"/>
-    <geometry>
-      <mesh filename="file://$(find hexapod_model_description)/meshes/femur_2_link_1.stl" scale="0.001 0.001 0.001"/>
-    </geometry>
-    <material name="silver"/>
-  </visual>
-  <collision>
-    <origin xyz="0.149643 -0.061207 -0.000912" rpy="0 0 0"/>
-    <geometry>
-      <mesh filename="file://$(find hexapod_model_description)/meshes/femur_2_link_1.stl" scale="0.001 0.001 0.001"/>
-    </geometry>
-  </collision>
-</link>
-<link name="coxa_2_link_1">
-  <inertial>
-    <origin xyz="-0.02599770016394727 -0.025997700307203414 -0.010119187749198275" rpy="0 0 0"/>
-    <mass value="0.36752045333400934"/>
-    <inertia ixx="0.000165" iyy="0.000165" izz="0.000292" ixy="-3e-05" iyz="-2e-05" ixz="-2e-05"/>
-  </inertial>
-  <visual>
-    <origin xyz="0.107782 -0.103068 -0.013762" rpy="0 0 0"/>
-    <geometry>
-      <mesh filename="file://$(find hexapod_model_description)/meshes/coxa_2_link_1.stl" scale="0.001 0.001 0.001"/>
-    </geometry>
-    <material name="silver"/>
-  </visual>
-  <collision>
-    <origin xyz="0.107782 -0.103068 -0.013762" rpy="0 0 0"/>
-    <geometry>
-      <mesh filename="file://$(find hexapod_model_description)/meshes/coxa_2_link_1.stl" scale="0.001 0.001 0.001"/>
-    </geometry>
-  </collision>
-</link>
-<link name="tibia_3_link_1">
-  <inertial>
-    <origin xyz="-0.04438810913290109 0.04423621896643121 3.191642993887996e-07" rpy="0 0 0"/>
-    <mass value="0.6509579807539126"/>
-    <inertia ixx="0.00103" iyy="0.000998" izz="0.001984" ixy="0.000792" iyz="0.0" ixz="-0.0"/>
-  </inertial>
-  <visual>
-    <origin xyz="0.217101 -0.374951 -0.000912" rpy="0 0 0"/>
-    <geometry>
-      <mesh filename="file://$(find hexapod_model_description)/meshes/tibia_3_link_1.stl" scale="0.001 0.001 0.001"/>
-    </geometry>
-    <material name="silver"/>
-  </visual>
-  <collision>
-    <origin xyz="0.217101 -0.374951 -0.000912" rpy="0 0 0"/>
-    <geometry>
-      <mesh filename="file://$(find hexapod_model_description)/meshes/tibia_3_link_1.stl" scale="0.001 0.001 0.001"/>
-    </geometry>
-  </collision>
-</link>
-<link name="femur_3_link_1">
-  <inertial>
-    <origin xyz="-0.03372863930509107 0.03372863916204971 3.1916430001611897e-07" rpy="0 0 0"/>
-    <mass value="1.2425883897057017"/>
-    <inertia ixx="0.000947" iyy="0.000947" izz="0.001691" ixy="0.000627" iyz="0.0" ixz="-0.0"/>
-  </inertial>
-  <visual>
-    <origin xyz="0.149643 -0.307493 -0.000912" rpy="0 0 0"/>
-    <geometry>
-      <mesh filename="file://$(find hexapod_model_description)/meshes/femur_3_link_1.stl" scale="0.001 0.001 0.001"/>
-    </geometry>
-    <material name="silver"/>
-  </visual>
-  <collision>
-    <origin xyz="0.149643 -0.307493 -0.000912" rpy="0 0 0"/>
-    <geometry>
-      <mesh filename="file://$(find hexapod_model_description)/meshes/femur_3_link_1.stl" scale="0.001 0.001 0.001"/>
-    </geometry>
-  </collision>
-</link>
-<link name="coxa_3_link_1">
-  <inertial>
-    <origin xyz="-0.0259977001641626 0.02599770002090629 -0.010119187749198146" rpy="0 0 0"/>
-    <mass value="0.36752045333400934"/>
-    <inertia ixx="0.000165" iyy="0.000165" izz="0.000292" ixy="3e-05" iyz="2e-05" ixz="-2e-05"/>
-  </inertial>
-  <visual>
-    <origin xyz="0.107782 -0.265632 -0.013762" rpy="0 0 0"/>
-    <geometry>
-      <mesh filename="file://$(find hexapod_model_description)/meshes/coxa_3_link_1.stl" scale="0.001 0.001 0.001"/>
-    </geometry>
-    <material name="silver"/>
-  </visual>
-  <collision>
-    <origin xyz="0.107782 -0.265632 -0.013762" rpy="0 0 0"/>
-    <geometry>
-      <mesh filename="file://$(find hexapod_model_description)/meshes/coxa_3_link_1.stl" scale="0.001 0.001 0.001"/>
-    </geometry>
-  </collision>
-</link>
-<link name="tibia_4_link_1">
-  <inertial>
-    <origin xyz="-0.00010740246556075264 0.06266738253711773 3.191642990343739e-07" rpy="0 0 0"/>
-    <mass value="0.6509579807539126"/>
-    <inertia ixx="0.001806" iyy="0.000223" izz="0.001984" ixy="-1.6e-05" iyz="0.0" ixz="0.0"/>
-  </inertial>
-  <visual>
-    <origin xyz="0.0265 -0.4539 -0.000912" rpy="0 0 0"/>
-    <geometry>
-      <mesh filename="file://$(find hexapod_model_description)/meshes/tibia_4_link_1.stl" scale="0.001 0.001 0.001"/>
-    </geometry>
-    <material name="silver"/>
-  </visual>
-  <collision>
-    <origin xyz="0.0265 -0.4539 -0.000912" rpy="0 0 0"/>
-    <geometry>
-      <mesh filename="file://$(find hexapod_model_description)/meshes/tibia_4_link_1.stl" scale="0.001 0.001 0.001"/>
-    </geometry>
-  </collision>
-</link>
-<link name="femur_4_link_1">
-  <inertial>
-    <origin xyz="-3.469446951953614e-18 0.047699999713918695 3.191642998002543e-07" rpy="0 0 0"/>
-    <mass value="1.2425883897057017"/>
-    <inertia ixx="0.001575" iyy="0.00032" izz="0.001691" ixy="0.0" iyz="0.0" ixz="-0.0"/>
-  </inertial>
-  <visual>
-    <origin xyz="0.0265 -0.3585 -0.000912" rpy="0 0 0"/>
-    <geometry>
-      <mesh filename="file://$(find hexapod_model_description)/meshes/femur_4_link_1.stl" scale="0.001 0.001 0.001"/>
-    </geometry>
-    <material name="silver"/>
-  </visual>
-  <collision>
-    <origin xyz="0.0265 -0.3585 -0.000912" rpy="0 0 0"/>
-    <geometry>
-      <mesh filename="file://$(find hexapod_model_description)/meshes/femur_4_link_1.stl" scale="0.001 0.001 0.001"/>
-    </geometry>
-  </collision>
-</link>
-<link name="coxa_4_link_1">
-  <inertial>
-    <origin xyz="-1.5211790160840621e-13 0.03676640679628457 -0.010119187749198275" rpy="0 0 0"/>
-    <mass value="0.36752045333400934"/>
-    <inertia ixx="0.000195" iyy="0.000135" izz="0.000292" ixy="-0.0" iyz="2.8e-05" ixz="-0.0"/>
-  </inertial>
-  <visual>
-    <origin xyz="0.0265 -0.2993 -0.013762" rpy="0 0 0"/>
-    <geometry>
-      <mesh filename="file://$(find hexapod_model_description)/meshes/coxa_4_link_1.stl" scale="0.001 0.001 0.001"/>
-    </geometry>
-    <material name="silver"/>
-  </visual>
-  <collision>
-    <origin xyz="0.0265 -0.2993 -0.013762" rpy="0 0 0"/>
-    <geometry>
-      <mesh filename="file://$(find hexapod_model_description)/meshes/coxa_4_link_1.stl" scale="0.001 0.001 0.001"/>
-    </geometry>
-  </collision>
-</link>
-<link name="tibia_5_link_1">
-  <inertial>
-    <origin xyz="0.0442362191094724 0.04438810898985973 3.1916429897083966e-07" rpy="0 0 0"/>
-    <mass value="0.6509579807539126"/>
-    <inertia ixx="0.000998" iyy="0.00103" izz="0.001984" ixy="-0.000792" iyz="0.0" ixz="0.0"/>
-  </inertial>
-  <visual>
-    <origin xyz="-0.164101 -0.374951 -0.000912" rpy="0 0 0"/>
-    <geometry>
-      <mesh filename="file://$(find hexapod_model_description)/meshes/tibia_5_link_1.stl" scale="0.001 0.001 0.001"/>
-    </geometry>
-    <material name="silver"/>
-  </visual>
-  <collision>
-    <origin xyz="-0.164101 -0.374951 -0.000912" rpy="0 0 0"/>
-    <geometry>
-      <mesh filename="file://$(find hexapod_model_description)/meshes/tibia_5_link_1.stl" scale="0.001 0.001 0.001"/>
-    </geometry>
-  </collision>
-</link>
-<link name="femur_5_link_1">
-  <inertial>
-    <origin xyz="0.03372863930509079 0.03372863916204982 3.1916429977672713e-07" rpy="0 0 0"/>
-    <mass value="1.2425883897057017"/>
-    <inertia ixx="0.000947" iyy="0.000947" izz="0.001691" ixy="-0.000627" iyz="0.0" ixz="0.0"/>
-  </inertial>
-  <visual>
-    <origin xyz="-0.096643 -0.307493 -0.000912" rpy="0 0 0"/>
-    <geometry>
-      <mesh filename="file://$(find hexapod_model_description)/meshes/femur_5_link_1.stl" scale="0.001 0.001 0.001"/>
-    </geometry>
-    <material name="silver"/>
-  </visual>
-  <collision>
-    <origin xyz="-0.096643 -0.307493 -0.000912" rpy="0 0 0"/>
-    <geometry>
-      <mesh filename="file://$(find hexapod_model_description)/meshes/femur_5_link_1.stl" scale="0.001 0.001 0.001"/>
-    </geometry>
-  </collision>
-</link>
-<link name="coxa_5_link_1">
-  <inertial>
-    <origin xyz="0.0259977001639473 0.02599770002112145 -0.010119187749198275" rpy="0 0 0"/>
-    <mass value="0.36752045333400934"/>
-    <inertia ixx="0.000165" iyy="0.000165" izz="0.000292" ixy="-3e-05" iyz="2e-05" ixz="2e-05"/>
-  </inertial>
-  <visual>
-    <origin xyz="-0.054782 -0.265632 -0.013762" rpy="0 0 0"/>
-    <geometry>
-      <mesh filename="file://$(find hexapod_model_description)/meshes/coxa_5_link_1.stl" scale="0.001 0.001 0.001"/>
-    </geometry>
-    <material name="silver"/>
-  </visual>
-  <collision>
-    <origin xyz="-0.054782 -0.265632 -0.013762" rpy="0 0 0"/>
-    <geometry>
-      <mesh filename="file://$(find hexapod_model_description)/meshes/coxa_5_link_1.stl" scale="0.001 0.001 0.001"/>
-    </geometry>
-  </collision>
-</link>
-<link name="tibia_6_link_1">
-  <inertial>
-    <origin xyz="0.0443881091329007 -0.04423621925251339 3.1916429900401624e-07" rpy="0 0 0"/>
-    <mass value="0.6509579807539126"/>
-    <inertia ixx="0.00103" iyy="0.000998" izz="0.001984" ixy="0.000792" iyz="-0.0" ixz="0.0"/>
-  </inertial>
-  <visual>
-    <origin xyz="-0.164101 0.006251 -0.000912" rpy="0 0 0"/>
-    <geometry>
-      <mesh filename="file://$(find hexapod_model_description)/meshes/tibia_6_link_1.stl" scale="0.001 0.001 0.001"/>
-    </geometry>
-    <material name="silver"/>
-  </visual>
-  <collision>
-    <origin xyz="-0.164101 0.006251 -0.000912" rpy="0 0 0"/>
-    <geometry>
-      <mesh filename="file://$(find hexapod_model_description)/meshes/tibia_6_link_1.stl" scale="0.001 0.001 0.001"/>
-    </geometry>
-  </collision>
-</link>
-<link name="femur_6_link_1">
-  <inertial>
-    <origin xyz="0.03372863930509079 -0.0337286394481318 3.1916429977672713e-07" rpy="0 0 0"/>
-    <mass value="1.2425883897057017"/>
-    <inertia ixx="0.000947" iyy="0.000947" izz="0.001691" ixy="0.000627" iyz="-0.0" ixz="0.0"/>
-  </inertial>
-  <visual>
-    <origin xyz="-0.096643 -0.061207 -0.000912" rpy="0 0 0"/>
-    <geometry>
-      <mesh filename="file://$(find hexapod_model_description)/meshes/femur_6_link_1.stl" scale="0.001 0.001 0.001"/>
-    </geometry>
-    <material name="silver"/>
-  </visual>
-  <collision>
-    <origin xyz="-0.096643 -0.061207 -0.000912" rpy="0 0 0"/>
-    <geometry>
-      <mesh filename="file://$(find hexapod_model_description)/meshes/femur_6_link_1.stl" scale="0.001 0.001 0.001"/>
-    </geometry>
-  </collision>
-</link>
-<link name="coxa_6_link_1">
-  <inertial>
-    <origin xyz="0.025997700164162404 -0.02599770030698831 -0.010119187749198275" rpy="0 0 0"/>
-    <mass value="0.36752045333400934"/>
-    <inertia ixx="0.000165" iyy="0.000165" izz="0.000292" ixy="3e-05" iyz="-2e-05" ixz="2e-05"/>
-  </inertial>
-  <visual>
-    <origin xyz="-0.054782 -0.103068 -0.013762" rpy="0 0 0"/>
-    <geometry>
-      <mesh filename="file://$(find hexapod_model_description)/meshes/coxa_6_link_1.stl" scale="0.001 0.001 0.001"/>
-    </geometry>
-    <material name="silver"/>
-  </visual>
-  <collision>
-    <origin xyz="-0.054782 -0.103068 -0.013762" rpy="0 0 0"/>
-    <geometry>
-      <mesh filename="file://$(find hexapod_model_description)/meshes/coxa_6_link_1.stl" scale="0.001 0.001 0.001"/>
-    </geometry>
-  </collision>
-</link>
-<joint name="tibia_1_joint" type="continuous">
-  <origin xyz="0.0 -0.0954 0.0" rpy="0 0 0"/>
-  <parent link="femur_1_link_1"/>
-  <child link="tibia_1_link_1"/>
-  <axis xyz="-1.0 0.0 -0.0"/>
-</joint>
-<joint name="femur_1_joint" type="continuous">
-  <origin xyz="0.0 -0.0592 -0.01285" rpy="0 0 0"/>
-  <parent link="coxa_1_link_1"/>
-  <child link="femur_1_link_1"/>
-  <axis xyz="-1.0 0.0 -0.0"/>
-</joint>
-<joint name="coxa_1_joint" type="continuous">
-  <origin xyz="-0.0265 0.0694 0.013762" rpy="0 0 0"/>
-  <parent link="base_link"/>
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