Commit message: Refactor hexapod URDF files: move transmissions to a separate file and update gazebo configuration

File: hexapod/urdf/hexapod_base.xacro (robot description, xacro)
@@ -489,190 +489,5 @@
   <axis xyz="0.0 0.0 1.0"/>
 </joint>
-<!-- Transmissions for all joints -->
-<!-- Leg 1 Transmissions -->
-<transmission name="coxa_1_transmission">
-  <type>transmission_interface/SimpleTransmission</type>
-  <joint name="coxa_1_joint">
-    <hardwareInterface>hardware_interface/PositionJointInterface</hardwareInterface>
-  </joint>
-  <actuator name="coxa_1_motor">
-    <hardwareInterface>hardware_interface/PositionJointInterface</hardwareInterface>
-    <mechanicalReduction>1</mechanicalReduction>
-  </actuator>
-</transmission>
-<transmission name="femur_1_transmission">
-  <type>transmission_interface/SimpleTransmission</type>
-  <joint name="femur_1_joint">
-    <hardwareInterface>hardware_interface/PositionJointInterface</hardwareInterface>
-  </joint>
-  <actuator name="femur_1_motor">
-    <hardwareInterface>hardware_interface/PositionJointInterface</hardwareInterface>
-    <mechanicalReduction>1</mechanicalReduction>
-  </actuator>
-</transmission>
-<transmission name="tibia_1_transmission">
-  <type>transmission_interface/SimpleTransmission</type>
-  <joint name="tibia_1_joint">
-    <hardwareInterface>hardware_interface/PositionJointInterface</hardwareInterface>
-  </joint>
-  <actuator name="tibia_1_motor">
-    <hardwareInterface>hardware_interface/PositionJointInterface</hardwareInterface>
-    <mechanicalReduction>1</mechanicalReduction>
-  </actuator>
-</transmission>
-<!-- Leg 2 Transmissions -->
-<transmission name="coxa_2_transmission">
-  <type>transmission_interface/SimpleTransmission</type>
-  <joint name="coxa_2_joint">
-    <hardwareInterface>hardware_interface/PositionJointInterface</hardwareInterface>
-  </joint>
-  <actuator name="coxa_2_motor">
-    <hardwareInterface>hardware_interface/PositionJointInterface</hardwareInterface>
-    <mechanicalReduction>1</mechanicalReduction>
-  </actuator>
-</transmission>
-<transmission name="femur_2_transmission">
-  <type>transmission_interface/SimpleTransmission</type>
-  <joint name="femur_2_joint">
-    <hardwareInterface>hardware_interface/PositionJointInterface</hardwareInterface>
-  </joint>
-  <actuator name="femur_2_motor">
-    <hardwareInterface>hardware_interface/PositionJointInterface</hardwareInterface>
-    <mechanicalReduction>1</mechanicalReduction>
-  </actuator>
-</transmission>
-<transmission name="tibia_2_transmission">
-  <type>transmission_interface/SimpleTransmission</type>
-  <joint name="tibia_2_joint">
-    <hardwareInterface>hardware_interface/PositionJointInterface</hardwareInterface>
-  </joint>
-  <actuator name="tibia_2_motor">
-    <hardwareInterface>hardware_interface/PositionJointInterface</hardwareInterface>
-    <mechanicalReduction>1</mechanicalReduction>
-  </actuator>
-</transmission>
-<!-- Leg 3 Transmissions -->
-<transmission name="coxa_3_transmission">
-  <type>transmission_interface/SimpleTransmission</type>
-  <joint name="coxa_3_joint">
-    <hardwareInterface>hardware_interface/PositionJointInterface</hardwareInterface>
-  </joint>
-  <actuator name="coxa_3_motor">
-    <hardwareInterface>hardware_interface/PositionJointInterface</hardwareInterface>
-    <mechanicalReduction>1</mechanicalReduction>
-  </actuator>
-</transmission>
-<transmission name="femur_3_transmission">
-  <type>transmission_interface/SimpleTransmission</type>
-  <joint name="femur_3_joint">
-    <hardwareInterface>hardware_interface/PositionJointInterface</hardwareInterface>
-  </joint>
-  <actuator name="femur_3_motor">
-    <hardwareInterface>hardware_interface/PositionJointInterface</hardwareInterface>
-    <mechanicalReduction>1</mechanicalReduction>
-  </actuator>
-</transmission>
-<transmission name="tibia_3_transmission">
-  <type>transmission_interface/SimpleTransmission</type>
-  <joint name="tibia_3_joint">
-    <hardwareInterface>hardware_interface/PositionJointInterface</hardwareInterface>
-  </joint>
-  <actuator name="tibia_3_motor">
-    <hardwareInterface>hardware_interface/PositionJointInterface</hardwareInterface>
-    <mechanicalReduction>1</mechanicalReduction>
-  </actuator>
-</transmission>
-<!-- Leg 4 Transmissions -->
-<transmission name="coxa_4_transmission">
-  <type>transmission_interface/SimpleTransmission</type>
-  <joint name="coxa_4_joint">
-    <hardwareInterface>hardware_interface/PositionJointInterface</hardwareInterface>
-  </joint>
-  <actuator name="coxa_4_motor">
-    <hardwareInterface>hardware_interface/PositionJointInterface</hardwareInterface>
-    <mechanicalReduction>1</mechanicalReduction>
-  </actuator>
-</transmission>
-<transmission name="femur_4_transmission">
-  <type>transmission_interface/SimpleTransmission</type>
-  <joint name="femur_4_joint">
-    <hardwareInterface>hardware_interface/PositionJointInterface</hardwareInterface>
-  </joint>
-  <actuator name="femur_4_motor">
-    <hardwareInterface>hardware_interface/PositionJointInterface</hardwareInterface>
-    <mechanicalReduction>1</mechanicalReduction>
-  </actuator>
-</transmission>
-<transmission name="tibia_4_transmission">
-  <type>transmission_interface/SimpleTransmission</type>
-  <joint name="tibia_4_joint">
-    <hardwareInterface>hardware_interface/PositionJointInterface</hardwareInterface>
-  </joint>
-  <actuator name="tibia_4_motor">
-    <hardwareInterface>hardware_interface/PositionJointInterface</hardwareInterface>
-    <mechanicalReduction>1</mechanicalReduction>
-  </actuator>
-</transmission>
-<!-- Leg 5 Transmissions -->
-<transmission name="coxa_5_transmission">
-  <type>transmission_interface/SimpleTransmission</type>
-  <joint name="coxa_5_joint">
-    <hardwareInterface>hardware_interface/PositionJointInterface</hardwareInterface>
-  </joint>
-  <actuator name="coxa_5_motor">
-    <hardwareInterface>hardware_interface/PositionJointInterface</hardwareInterface>
-    <mechanicalReduction>1</mechanicalReduction>
-  </actuator>
-</transmission>
-<transmission name="femur_5_transmission">
-  <type>transmission_interface/SimpleTransmission</type>
-  <joint name="femur_5_joint">
-    <hardwareInterface>hardware_interface/PositionJointInterface</hardwareInterface>
-  </joint>
-  <actuator name="femur_5_motor">
-    <hardwareInterface>hardware_interface/PositionJointInterface</hardwareInterface>
-    <mechanicalReduction>1</mechanicalReduction>
-  </actuator>
-</transmission>
-<transmission name="tibia_5_transmission">
-  <type>transmission_interface/SimpleTransmission</type>
-  <joint name="tibia_5_joint">
-    <hardwareInterface>hardware_interface/PositionJointInterface</hardwareInterface>
-  </joint>
-  <actuator name="tibia_5_motor">
-    <hardwareInterface>hardware_interface/PositionJointInterface</hardwareInterface>
-    <mechanicalReduction>1</mechanicalReduction>
-  </actuator>
-</transmission>
-<!-- Leg 6 Transmissions -->
-<transmission name="coxa_6_transmission">
-  <type>transmission_interface/SimpleTransmission</type>
-  <joint name="coxa_6_joint">
-    <hardwareInterface>hardware_interface/PositionJointInterface</hardwareInterface>
-  </joint>
-  <actuator name="coxa_6_motor">
-    <hardwareInterface>hardware_interface/PositionJointInterface</hardwareInterface>
-    <mechanicalReduction>1</mechanicalReduction>
-  </actuator>
-</transmission>
-<transmission name="femur_6_transmission">
-  <type>transmission_interface/SimpleTransmission</type>
-  <joint name="femur_6_joint">
-    <hardwareInterface>hardware_interface/PositionJointInterface</hardwareInterface>
-  </joint>
-  <actuator name="femur_6_motor">
-    <hardwareInterface>hardware_interface/PositionJointInterface</hardwareInterface>
-    <mechanicalReduction>1</mechanicalReduction>
-  </actuator>
-</transmission>
-<transmission name="tibia_6_transmission">
-  <type>transmission_interface/SimpleTransmission</type>
-  <joint name="tibia_6_joint">
-    <hardwareInterface>hardware_interface/PositionJointInterface</hardwareInterface>
-  </joint>
-  <actuator name="tibia_6_motor">
-    <hardwareInterface>hardware_interface/PositionJointInterface</hardwareInterface>
-    <mechanicalReduction>1</mechanicalReduction>
-  </actuator>
-</transmission>
+<!-- Include transmissions from separate file -->
+<xacro:include filename="hexapod_transmissions.xacro"/>
 </robot>

File: hexapod/urdf/hexapod_base_gazebo.xacro (robot description, xacro)
@@ -1,4 +1,4 @@
 <?xml version="1.0" ?>
-<robot xmlns:xacro="http://www.ros.org/wiki/xacro" >
+<robot name="hexapod" xmlns:xacro="http://www.ros.org/wiki/xacro">
     <!-- Gazebo ros2_control plugin -->
     <gazebo>
@@ -6,5 +6,4 @@
             <robot_param>robot_description</robot_param>
             <robot_param_node>robot_state_publisher</robot_param_node>
-            <parameters>$(find hexapod_control)/config/hexapod_controllers.yaml</parameters>
         </plugin>
     </gazebo>
@@ -49,4 +48,5 @@
         <hardware>
             <plugin>gz_ros2_control/GzSystem</plugin>
+            <param name="update_rate">100</param>
         </hardware>
         <!-- Joint interfaces for all legs -->
