Commit message: Refactor hexapod control configuration for clarity and consistency

File: hexapod_model_description/control/hexapod.ros2_control.xacro (robot description, xacro)
@@ -56,134 +56,134 @@
             <!-- Each leg has 3 joints for 18 total actuated joints                -->
             <!-- Leg 1 joints (Front-right leg) -->
-            <joint name="joint1_1">
-                <command_interface name="position"/>  <!-- controlling joint positions -->
-                <state_interface name="position">
-                  <param name="initial_value">${initial_positions['joint1_1']}</param> <!-- Configuring initial value -->
-                </state_interface>
-                <state_interface name="velocity"/>
+            <joint name="coxa_joint_1">
+              <command_interface name="position"/>
+              <state_interface name="position">
+                <param name="initial_value">${initial_positions['coxa_joint_1']}</param>
+              </state_interface>
+              <state_interface name="velocity"/>
             </joint>
-            <joint name="joint2_1">
-                <command_interface name="position"/>
-                <state_interface name="position">
-                  <param name="initial_value">${initial_positions['joint2_1']}</param>
-                </state_interface>
-                <state_interface name="velocity"/>
+            <joint name="femur_joint_1">
+              <command_interface name="position"/>
+              <state_interface name="position">
+                <param name="initial_value">${initial_positions['femur_joint_1']}</param>
+              </state_interface>
+              <state_interface name="velocity"/>
             </joint>
-            <joint name="joint3_1">
-                <command_interface name="position"/>
-                <state_interface name="position">
-                  <param name="initial_value">${initial_positions['joint3_1']}</param>
-                </state_interface>
-                <state_interface name="velocity"/>
+            <joint name="tibia_joint_1">
+              <command_interface name="position"/>
+              <state_interface name="position">
+                <param name="initial_value">${initial_positions['tibia_joint_1']}</param>
+              </state_interface>
+              <state_interface name="velocity"/>
             </joint>
             <!-- Leg 2 joints (Middle-right leg) -->
-            <joint name="joint1_2">
-                <command_interface name="position"/>
-                <state_interface name="position">
-                  <param name="initial_value">${initial_positions['joint1_2']}</param>
-                </state_interface>
-                <state_interface name="velocity"/>
+            <joint name="coxa_joint_2">
+              <command_interface name="position"/>
+              <state_interface name="position">
+                <param name="initial_value">${initial_positions['coxa_joint_2']}</param>
+              </state_interface>
+              <state_interface name="velocity"/>
             </joint>
-            <joint name="joint2_2">
-                <command_interface name="position"/>
-                <state_interface name="position">
-                  <param name="initial_value">${initial_positions['joint2_2']}</param>
-                </state_interface>
-                <state_interface name="velocity"/>
+            <joint name="femur_joint_2">
+              <command_interface name="position"/>
+              <state_interface name="position">
+                <param name="initial_value">${initial_positions['femur_joint_2']}</param>
+              </state_interface>
+              <state_interface name="velocity"/>
             </joint>
-            <joint name="joint3_2">
-                <command_interface name="position"/>
-                <state_interface name="position">
-                  <param name="initial_value">${initial_positions['joint3_2']}</param>
-                </state_interface>
-                <state_interface name="velocity"/>
+            <joint name="tibia_joint_2">
+              <command_interface name="position"/>
+              <state_interface name="position">
+                <param name="initial_value">${initial_positions['tibia_joint_2']}</param>
+              </state_interface>
+              <state_interface name="velocity"/>
             </joint>
             <!-- Leg 3 joints (Rear-right leg) -->
-            <joint name="joint1_3">
-                <command_interface name="position"/>
-                <state_interface name="position">
-                  <param name="initial_value">${initial_positions['joint1_3']}</param>
-                </state_interface>
-                <state_interface name="velocity"/>
+            <joint name="coxa_joint_3">
+              <command_interface name="position"/>
+              <state_interface name="position">
+                <param name="initial_value">${initial_positions['coxa_joint_3']}</param>
+              </state_interface>
+              <state_interface name="velocity"/>
             </joint>
-            <joint name="joint2_3">
-                <command_interface name="position"/>
-                <state_interface name="position">
-                  <param name="initial_value">${initial_positions['joint2_3']}</param>
-                </state_interface>
-                <state_interface name="velocity"/>
+            <joint name="femur_joint_3">
+              <command_interface name="position"/>
+              <state_interface name="position">
+                <param name="initial_value">${initial_positions['femur_joint_3']}</param>
+              </state_interface>
+              <state_interface name="velocity"/>
             </joint>
-            <joint name="joint3_3">
-                <command_interface name="position"/>
-                <state_interface name="position">
-                  <param name="initial_value">${initial_positions['joint3_3']}</param>
-                </state_interface>
-                <state_interface name="velocity"/>
+            <joint name="tibia_joint_3">
+              <command_interface name="position"/>
+              <state_interface name="position">
+                <param name="initial_value">${initial_positions['tibia_joint_3']}</param>
+              </state_interface>
+              <state_interface name="velocity"/>
             </joint>
             <!-- Leg 4 joints (Rear-left leg) -->
-            <joint name="joint1_4">
-                <command_interface name="position"/>
-                <state_interface name="position">
-                  <param name="initial_value">${initial_positions['joint1_4']}</param>
-                </state_interface>
-                <state_interface name="velocity"/>
+            <joint name="coxa_joint_4">
+              <command_interface name="position"/>
+              <state_interface name="position">
+                <param name="initial_value">${initial_positions['coxa_joint_4']}</param>
+              </state_interface>
+              <state_interface name="velocity"/>
             </joint>
-            <joint name="joint2_4">
-                <command_interface name="position"/>
-                <state_interface name="position">
-                  <param name="initial_value">${initial_positions['joint2_4']}</param>
-                </state_interface>
-                <state_interface name="velocity"/>
+            <joint name="femur_joint_4">
+              <command_interface name="position"/>
+              <state_interface name="position">
+                <param name="initial_value">${initial_positions['femur_joint_4']}</param>
+              </state_interface>
+              <state_interface name="velocity"/>
             </joint>
-            <joint name="joint3_4">
-                <command_interface name="position"/>
-                <state_interface name="position">
-                  <param name="initial_value">${initial_positions['joint3_4']}</param>
-                </state_interface>
-                <state_interface name="velocity"/>
+            <joint name="tibia_joint_4">
+              <command_interface name="position"/>
+              <state_interface name="position">
+                <param name="initial_value">${initial_positions['tibia_joint_4']}</param>
+              </state_interface>
+              <state_interface name="velocity"/>
             </joint>
             <!-- Leg 5 joints (Middle-left leg) -->
-            <joint name="joint1_5">
-                <command_interface name="position"/>
-                <state_interface name="position">
-                  <param name="initial_value">${initial_positions['joint1_5']}</param>
-                </state_interface>
-                <state_interface name="velocity"/>
+            <joint name="coxa_joint_5">
+              <command_interface name="position"/>
+              <state_interface name="position">
+                <param name="initial_value">${initial_positions['coxa_joint_5']}</param>
+              </state_interface>
+              <state_interface name="velocity"/>
             </joint>
-            <joint name="joint2_5">
-                <command_interface name="position"/>
-                <state_interface name="position">
-                  <param name="initial_value">${initial_positions['joint2_5']}</param>
-                </state_interface>
-                <state_interface name="velocity"/>
+            <joint name="femur_joint_5">
+              <command_interface name="position"/>
+              <state_interface name="position">
+                <param name="initial_value">${initial_positions['femur_joint_5']}</param>
+              </state_interface>
+              <state_interface name="velocity"/>
             </joint>
-            <joint name="joint3_5">
-                <command_interface name="position"/>
-                <state_interface name="position">
-                  <param name="initial_value">${initial_positions['joint3_5']}</param>
-                </state_interface>
-                <state_interface name="velocity"/>
+            <joint name="tibia_joint_5">
+              <command_interface name="position"/>
+              <state_interface name="position">
+                <param name="initial_value">${initial_positions['tibia_joint_5']}</param>
+              </state_interface>
+              <state_interface name="velocity"/>
             </joint>
             <!-- Leg 6 joints (Front-left leg) -->
-            <joint name="joint1_6">
-                <command_interface name="position"/>
-                <state_interface name="position">
-                  <param name="initial_value">${initial_positions['joint1_6']}</param>
-                </state_interface>
-                <state_interface name="velocity"/>
+            <joint name="coxa_joint_6">
+              <command_interface name="position"/>
+              <state_interface name="position">
+                <param name="initial_value">${initial_positions['coxa_joint_6']}</param>
+              </state_interface>
+              <state_interface name="velocity"/>
             </joint>
-            <joint name="joint2_6">
-                <command_interface name="position"/>
-                <state_interface name="position">
-                  <param name="initial_value">${initial_positions['joint2_6']}</param>
-                </state_interface>
-                <state_interface name="velocity"/>
+            <joint name="femur_joint_6">
+              <command_interface name="position"/>
+              <state_interface name="position">
+                <param name="initial_value">${initial_positions['femur_joint_6']}</param>
+              </state_interface>
+              <state_interface name="velocity"/>
             </joint>
-            <joint name="joint3_6">
-                <command_interface name="position"/>
-                <state_interface name="position">
-                  <param name="initial_value">${initial_positions['joint3_6']}</param>
-                </state_interface>
-                <state_interface name="velocity"/>
+            <joint name="tibia_joint_6">
+              <command_interface name="position"/>
+              <state_interface name="position">
+                <param name="initial_value">${initial_positions['tibia_joint_6']}</param>
+              </state_interface>
+              <state_interface name="velocity"/>
             </joint>
         </ros2_control>
