Commit message: Update hexapod model configurations: adjust initial joint positions, enhance materials, and add LiDAR sensor plugin

File: hexapod_model_description/gazebo/hexapod.gazebo.xacro (robot description, xacro)
@@ -36,4 +36,39 @@
     </gazebo>
   </xacro:macro>
+  <!-- LiDAR/Laser Scanner Gazebo Plugin -->
+  <gazebo reference="laser_link">
+    <sensor type="gpu_lidar" name="laser">
+      <update_rate>10</update_rate>
+      <pose>0 0 0 0 0 0</pose>
+      <ray>
+        <scan>
+          <horizontal>
+            <samples>720</samples>
+            <resolution>1</resolution>
+            <min_angle>-1.5708</min_angle>
+            <max_angle>1.5708</max_angle>
+          </horizontal>
+        </scan>
+        <range>
+          <min>0.12</min>
+          <max>10.0</max>
+          <resolution>0.01</resolution>
+        </range>
+        <noise>
+          <type>gaussian</type>
+          <mean>0.0</mean>
+          <stddev>0.01</stddev>
+        </noise>
+      </ray>
+      <plugin name="gz_lidar_plugin" filename="libgz_ros2_laser_scan.so">
+        <ros>
+          <namespace></namespace>
+          <remapping>~/out:=scan</remapping>
+        </ros>
+        <frame_name>laser_link</frame_name>
+      </plugin>
+    </sensor>
+    <material>Gazebo/Red</material>
+  </gazebo>
   <!-- GAZEBO REFERENCES FOR ALL ROBOT LINKS                            -->
   <!-- Main physics parameters applied to platform -->

File: hexapod_model_description/urdf/hexapod_leg_ee.urdf.xacro (robot description, xacro)
@@ -349,6 +349,6 @@
             <mesh filename="file://$(find hexapod_model_description)/meshes/${prefix}_link.stl" scale="0.001 0.001 0.001"/>
           </geometry>
-          <material name="gray">
-            <color rgba="0.2 0.2 0.2 1"/>
+          <material name="black">
+            <color rgba="0.1 0.1 0.1 1"/>
           </material>
         </visual>
@@ -375,7 +375,14 @@
             <mesh filename="file://$(find hexapod_model_description)/meshes/${prefix}_${index}_link.stl" scale="0.001 0.001 0.001"/>
           </geometry>
-          <material name="grey">
-            <color rgba="${rgba}"/>
-          </material>
+          <xacro:if value="${prefix == 'femur'}">
+            <material name="orange">
+              <color rgba="1.0 0.4 0.0 1"/>
+            </material>
+          </xacro:if>
+          <xacro:unless value="${prefix == 'femur'}">
+            <material name="black">
+              <color rgba="0.1 0.1 0.1 1"/>
+            </material>
+          </xacro:unless>
         </visual>
         <collision>
@@ -410,5 +417,5 @@
       <xacro:base
       prefix="base"
-      rgba="0.2 0.2 0.2 1"
+      rgba="0.1 0.1 0.1 1"
       mass="${base_mass}"
       c_xyz="${base_c_xyz}"
@@ -434,5 +441,5 @@
       i_xyz="${coxa_1_i_xyz}"
       i_rpy="${coxa_1_i_rpy}"
-      rgba="0.2 0.2 0.2 1"
+      rgba="0.1 0.1 0.1 1"
       mass="${coxa_mass}"
       ixx="${coxa_1_ixx}"
@@ -462,5 +469,5 @@
       i_xyz="${femur_1_i_xyz}"
       i_rpy="${femur_1_i_rpy}"
-      rgba="0.2 0.2 0.2 1"
+      rgba="1.0 0.4 0.0 1"
       mass="${femur_mass}"
       ixx="${femur_1_ixx}"
@@ -490,5 +497,5 @@
       i_xyz="${tibia_1_i_xyz}"
       i_rpy="${tibia_1_i_rpy}"
-      rgba="0.2 0.2 0.2 1"
+      rgba="0.1 0.1 0.1 1"
       mass="${tibia_mass}"
       ixx="${tibia_1_ixx}"
@@ -519,5 +526,5 @@
       i_xyz="${coxa_2_i_xyz}"
       i_rpy="${coxa_2_i_rpy}"
-      rgba="0.2 0.2 0.2 1"
+      rgba="0.1 0.1 0.1 1"
       mass="${coxa_mass}"
       ixx="${coxa_2_ixx}"
@@ -547,5 +554,5 @@
       i_xyz="${femur_2_i_xyz}"
       i_rpy="${femur_2_i_rpy}"
-      rgba="0.2 0.2 0.2 1"
+      rgba="1.0 0.4 0.0 1"
       mass="${femur_mass}"
       ixx="${femur_2_ixx}"
@@ -575,5 +582,5 @@
       i_xyz="${tibia_2_i_xyz}"
       i_rpy="${tibia_2_i_rpy}"
-      rgba="0.2 0.2 0.2 1"
+      rgba="0.1 0.1 0.1 1"
       mass="${tibia_mass}"
       ixx="${tibia_2_ixx}"
@@ -604,5 +611,5 @@
       i_xyz="${coxa_3_i_xyz}"
       i_rpy="${coxa_3_i_rpy}"
-      rgba="0.2 0.2 0.2 1"
+      rgba="0.1 0.1 0.1 1"
       mass="${coxa_mass}"
       ixx="${coxa_3_ixx}"
@@ -632,5 +639,5 @@
       i_xyz="${femur_3_i_xyz}"
       i_rpy="${femur_3_i_rpy}"
-      rgba="0.2 0.2 0.2 1"
+      rgba="1.0 0.4 0.0 1"
       mass="${femur_mass}"
       ixx="${femur_3_ixx}"
@@ -660,5 +667,5 @@
       i_xyz="${tibia_3_i_xyz}"
       i_rpy="${tibia_3_i_rpy}"
-      rgba="0.2 0.2 0.2 1"
+      rgba="0.1 0.1 0.1 1"
       mass="${tibia_mass}"
       ixx="${tibia_3_ixx}"
@@ -689,5 +696,5 @@
       i_xyz="${coxa_4_i_xyz}"
       i_rpy="${coxa_4_i_rpy}"
-      rgba="0.2 0.2 0.2 1"
+      rgba="0.1 0.1 0.1 1"
       mass="${coxa_mass}"
       ixx="${coxa_4_ixx}"
@@ -717,5 +724,5 @@
       i_xyz="${femur_4_i_xyz}"
       i_rpy="${femur_4_i_rpy}"
-      rgba="0.2 0.2 0.2 1"
+      rgba="1.0 0.4 0.0 1"
       mass="${femur_mass}"
       ixx="${femur_4_ixx}"
@@ -745,5 +752,5 @@
       i_xyz="${tibia_4_i_xyz}"
       i_rpy="${tibia_4_i_rpy}"
-      rgba="0.2 0.2 0.2 1"
+      rgba="0.1 0.1 0.1 1"
       mass="${tibia_mass}"
       ixx="${tibia_4_ixx}"
@@ -774,5 +781,5 @@
       i_xyz="${coxa_5_i_xyz}"
       i_rpy="${coxa_5_i_rpy}"
-      rgba="0.2 0.2 0.2 1"
+      rgba="0.1 0.1 0.1 1"
       mass="${coxa_mass}"
       ixx="${coxa_5_ixx}"
@@ -802,5 +809,5 @@
       i_xyz="${femur_5_i_xyz}"
       i_rpy="${femur_5_i_rpy}"
-      rgba="0.2 0.2 0.2 1"
+      rgba="1.0 0.4 0.0 1"
       mass="${femur_mass}"
       ixx="${femur_5_ixx}"
@@ -830,5 +837,5 @@
       i_xyz="${tibia_5_i_xyz}"
       i_rpy="${tibia_5_i_rpy}"
-      rgba="0.2 0.2 0.2 1"
+      rgba="0.1 0.1 0.1 1"
       mass="${tibia_mass}"
       ixx="${tibia_5_ixx}"
@@ -859,5 +866,5 @@
       i_xyz="${coxa_6_i_xyz}"
       i_rpy="${coxa_6_i_rpy}"
-      rgba="0.2 0.2 0.2 1"
+      rgba="0.1 0.1 0.1 1"
       mass="${coxa_mass}"
       ixx="${coxa_6_ixx}"
@@ -887,5 +894,5 @@
       i_xyz="${femur_6_i_xyz}"
       i_rpy="${femur_6_i_rpy}"
-      rgba="0.2 0.2 0.2 1"
+      rgba="1.0 0.4 0.0 1"
       mass="${femur_mass}"
       ixx="${femur_6_ixx}"
@@ -915,5 +922,5 @@
       i_xyz="${tibia_6_i_xyz}"
       i_rpy="${tibia_6_i_rpy}"
-      rgba="0.2 0.2 0.2 1"
+      rgba="0.1 0.1 0.1 1"
       mass="${tibia_mass}"
       ixx="${tibia_6_ixx}"

File: hexapod_model_description/urdf/materials.xacro (robot description, xacro)
@@ -1,6 +1,6 @@
 <?xml version="1.0"?>
 <robot xmlns:xacro="http://www.ros.org/wiki/xacro">
-  <material name="white">
-    <color rgba="1 1 1 1"/>
+  <material name="orange">
+    <color rgba="1 0.624 0 1"/>
   </material>
   <material name="black">
